File: pcb_files/pcb_thesis/pcb_thesis_custom.kicad_pcb (KiCad board)
At the start: 2 copper layers, 23 parts, among them J1 goldpin 1x6, J2 goldpin 1x2, J3 goldpin 1x2, Q1 Q_PNP_BCE, SW1 RESET SW, SW2 POWER_SW, SW3 ACTION SW, U1 ATmega32L-8AU, Y1 8MHz

Commit message: pcb in progress
Parts:
- added J4: goldpin 1x2, Connector_PinHeader_2.54mm:PinHeader_1x02_P2.54mm_Horizontal, F.Cu at (203.0, 56.5)
- D3, D4: footprint Diode_SMD:D_SOT-23_NKA -> Package_TO_SOT_SMD:SOT-23_Handsoldering
- moved J3 101.4 mm to (146.5, 32.0), turned to 270 degrees
- moved Y1 91.5 mm to (189.5, 37.0), turned to 0 degrees
- moved D5 90.1 mm to (153.0, 37.0), turned to 90 degrees
- moved Q1 64.4 mm to (145.5, 48.5)
- moved D1 59.4 mm to (167.5, 51.0), turned to 0 degrees
- moved J1 57.9 mm to (203.0, 37.0)
- moved J2 57.9 mm to (203.0, 30.5)
- moved C3 54.9 mm to (173.0, 44.0), turned to 270 degrees
- moved D2 53.8 mm to (167.5, 48.0), turned to 0 degrees
- moved C4 53.4 mm to (169.0, 44.0), turned to 0 degrees
- moved C5 52.8 mm to (176.0, 41.0), turned to 0 degrees
- moved R2 52.3 mm to (163.5, 51.0)
- moved U1 51.7 mm to (181.0, 50.5)
- moved R3 51.2 mm to (163.5, 48.0)
- moved SW1 50.9 mm to (164.5, 60.0), turned to 0 degrees
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Connections:
- C3 pad 1: Net-(C3-Pad1) -> VCC
- C4 pad 2: Net-(C3-Pad1) -> VCC
- C5 pad 2: Net-(C3-Pad1) -> VCC
- D4 pad 1: Net-(D3-Pad3) -> Net-(D4-Pad1)
- J1 pad 1: GND -> /~RESET
- J1 pad 5: /~RESET -> /+5V_USBasp
- J1 pad 6: +5V -> GND
- Q1 pad 2: Net-(D3-Pad1) -> Net-(D4-Pad1)
- Q1 pad 3: +5V -> VCC
- R1 pad 1: +5V -> VCC
- SW2 pad 2: Net-(C3-Pad1) -> VCC
- SW2 pad 3: +5V -> /+5V_USBasp
- U1 pad 12: Net-(U1-Pad12) -> Net-(SW3-Pad1)
- U1 pad 17: Net-(C3-Pad1) -> VCC
- U1 pad 27: Net-(C3-Pad1) -> VCC
- U1 pad 36: Net-(SW3-Pad1) -> Net-(U1-Pad36)
- U1 pad 38: Net-(C3-Pad1) -> VCC
- U1 pad 5: Net-(C3-Pad1) -> VCC
Routing:
- net VCC: track 0.00 -> 156.0 mm
- net GND: track 0.00 -> 75.5 mm
- net /~RESET: track 0.00 -> 51.2 mm
- net Net-(J2-Pad1): track 0.00 -> 45.2 mm
- net Net-(J2-Pad2): track 0.00 -> 44.9 mm
- net Net-(SW3-Pad1): track 0.00 -> 36.5 mm
- net /M+: track 0.00 -> 26.6 mm
- net Net-(J1-Pad2): track 0.00 -> 21.8 mm
- net Net-(J1-Pad3): track 0.00 -> 21.1 mm
- net Net-(Q1-Pad1): track 0.00 -> 20.9 mm
- net Net-(J1-Pad4): track 0.00 -> 20.4 mm
- net Net-(C2-Pad2): track 0.00 -> 17.3 mm
- net Net-(C1-Pad2): track 0.00 -> 17.2 mm
- net /+5V_USBasp: track 0.00 -> 16.0 mm
- net Net-(D2-Pad2): track 0.00 -> 8.47 mm
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- added copper zone on F.Cu, net GND
Other:
- net class Default: trace_width 0.25 -> 0.5
- net class main05 added: clearance 0.2, trace_width 0.5, via_dia 0.8, via_drill 0.4
