File: pcb_files/pcb_thesis/pcb_thesis.sch (KiCad schematic (older format))
At the start: 21 parts

Commit message: updated schematic files to be more actual
Parts:
- added BT?: 9V, symbol Device:Battery_Cell
- added J?: goldpin 1x2, symbol Connector:Conn_01x02_Female
- added M?: Motor_DC, symbol Motor:Motor_DC
- added U?: LD1117S50TR_SOT223, Package_TO_SOT_SMD:SOT-223-3_TabPin2, symbol Regulator_Linear:LD1117S50TR_SOT223
- C? (x2): value C -> 22p
- C? (x2): value C -> 100n
- C?: value CP -> 22u
- J?: value Conn_01x04_Male -> goldpin 1x4
- J? (x2): value Conn_01x02_Male -> goldpin 1x2
- R?: value R -> 10k
- R? (x2): value R -> 370
- SW?: value SW_DPST_x2 -> RESET SW
- SW?: value SW_DPST_x2 -> ACTION SW
- Y?: value Crystal -> 8MHz
Connections:
- net labels added: +5VP
- wire segments 79 -> 96
Other:
- note added: "Silnik\nwibracyjny"
- note added: "USART"
- note added: "USBasp"
- moved on the sheet: D?, J?, Q?, SW?A

Commit message: updated pcb files
divided schematic into parts and discarded option with source of energy but schematic is prepared for this feature
Parts:
- removed BT?: 9V, symbol Device:Battery_Cell
- removed U?: ATmega32A-AU, Package_QFP:TQFP-44_10x10mm_P0.8mm, symbol MCU_Microchip_ATmega:ATmega32A-AU
- removed U?: LD1117S50TR_SOT223, Package_TO_SOT_SMD:SOT-223-3_TabPin2, symbol Regulator_Linear:LD1117S50TR_SOT223
- added SW?: SW_SPDT, symbol Switch:SW_SPDT
- added U?: ATmega32L-8AU, Package_QFP:TQFP-44_10x10mm_P0.8mm, symbol MCU_Microchip_ATmega:ATmega32L-8AU
Connections:
- net labels added: +BATT
- net labels removed: +5VP
- wire segments 96 -> 91
Changed lines of the file:
@@
 L power:+5V #PWR?
 U 1 1 5C463787
-P 4400 1750
-F 0 "#PWR?" H 4400 1600 50  0001 C CNN
-F 1 "+5V" H 4415 1923 50  0000 C CNN
-F 2 "" H 4400 1750 50  0001 C CNN
-F 3 "" H 4400 1750 50  0001 C CNN
-	1    4400 1750
+P 4500 1300
+F 0 "#PWR?" H 4500 1150 50  0001 C CNN
+F 1 "+5V" H 4500 1450 50  0000 C CNN
+F 2 "" H 4500 1300 50  0001 C CNN
+F 3 "" H 4500 1300 50  0001 C CNN
+	1    4500 1300
 	1    0    0    -1
 $EndComp
@@
 	-1   0    0    1
 $EndComp
-$Comp
-L MCU_Microchip_ATmega:ATmega32A-AU U?
-U 1 1 5C46225A
-P 5150 4050
-F 0 "U?" H 4700 2100 50  0000 C CNN
-F 1 "ATmega32A-AU" H 5500 2050 50  0000 C CNN
-F 2 "Package_QFP:TQFP-44_10x10mm_P0.8mm" H 5150 4050 50  0001 C CIN
-F 3 "http://ww1.microchip.com/downloads/en/DeviceDoc/atmel-8155-8-bit-microcontroller-avr-atmega32a_datasheet.pdf" H 5150 4050 50  0001 C CNN
-	1    5150 4050
-	1    0    0    -1
-$EndComp
 Wire Wire Line
 	5750 5050 6050 5050
@@
 NoConn ~ 5750 4650
 $Comp
-L Device:Battery_Cell BT?
-U 1 1 5CD7005F
-P 1750 4300
-F 0 "BT?" H 1868 4396 50  0000 L CNN
-F 1 "9V" H 1868 4305 50  0000 L CNN
-F 2 "" V 1750 4360 50  0001 C CNN
-F 3 "~" V 1750 4360 50  0001 C CNN
-	1    1750 4300
-	1    0    0    -1
-$EndComp
-$Comp
-L Regulator_Linear:LD1117S50TR_SOT223 U?
-U 1 1 5CD70646
-P 2700 3950
-F 0 "U?" H 2700 4192 50  0000 C CNN
-F 1 "LD1117S50TR_SOT223" H 2700 4101 50  0000 C CNN
-F 2 "Package_TO_SOT_SMD:SOT-223-3_TabPin2" H 2700 4150 50  0001 C CNN
-F 3 "http://www.st.com/st-web-ui/static/active/en/resource/technical/document/datasheet/CD00000544.pdf" H 2800 3700 50  0001 C CNN
-	1    2700 3950
-	1    0    0    -1
-$EndComp
-Wire Wire Line
-	1750 4100 1750 3950
-Wire Wire Line
-	1750 3950 2400 3950
-$Comp
-L power:GND #PWR?
-U 1 1 5CD7263D
-P 1750 4600
-F 0 "#PWR?" H 1750 4350 50  0001 C CNN
-F 1 "GND" H 1755 4427 50  0000 C CNN
-F 2 "" H 1750 4600 50  0001 C CNN
-F 3 "" H 1750 4600 50  0001 C CNN
-	1    1750 4600
-	1    0    0    -1
-$EndComp
-Wire Wire Line
-	1750 4600 1750 4450
-Wire Wire Line
-	2700 4250 2700 4450
-Wire Wire Line
-	2700 4450 1750 4450
-Connection ~ 1750 4450
-Wire Wire Line
-	1750 4450 1750 4400
-$Comp
-L power:+5VP #PWR?
-U 1 1 5CD76483
-P 3250 3850
-F 0 "#PWR?" H 3250 3700 50  0001 C CNN
-F 1 "+5VP" H 3265 4023 50  0000 C CNN
-F 2 "" H 3250 3850 50  0001 C CNN
-F 3 "" H 3250 3850 50  0001 C CNN
-	1    3250 3850
-	1    0    0    -1
-$EndComp
-Wire Wire Line
-	3000 3950 3250 3950
-Wire Wire Line
-	3250 3950 3250 3850
+L MCU_Microchip_ATmega:ATmega32L-8AU U?
+U 1 1 5CD8387E
+P 5150 4050
+F 0 "U?" H 4700 2000 50  0000 C CNN
+F 1 "ATmega32L-8AU" H 5550 2050 50  0000 C CNN
+F 2 "Package_QFP:TQFP-44_10x10mm_P0.8mm" H 5150 4050 50  0001 C CIN
+F 3 "http://ww1.microchip.com/downloads/en/DeviceDoc/doc2503.pdf" H 5150 4050 50  0001 C CNN
+	1    5150 4050
+	1    0    0    -1
+$EndComp
+$Comp
+L Switch:SW_SPDT SW?
+U 1 1 5CD848F9
+P 4400 1550
+F 0 "SW?" V 4446 1362 50  0000 R CNN
+F 1 "SW_SPDT" V 4355 1362 50  0000 R CNN
+F 2 "" H 4400 1550 50  0001 C CNN
+F 3 "" H 4400 1550 50  0001 C CNN
+	1    4400 1550
+	0    -1   -1   0
+$EndComp
+$Comp
+L power:+BATT #PWR?
+U 1 1 5CD86795
+P 4300 1300
+F 0 "#PWR?" H 4300 1150 50  0001 C CNN
+F 1 "+BATT" H 4250 1450 50  0000 C CNN
+F 2 "" H 4300 1300 50  0001 C CNN
+F 3 "" H 4300 1300 50  0001 C CNN
+	1    4300 1300
+	1    0    0    -1
+$EndComp
+Wire Wire Line
+	4300 1300 4300 1350
+Wire Wire Line
+	4500 1300 4500 1350
+$Comp
+L power:+BATT #PWR?
+U 1 1 5CD8A13B
+P 1400 1950
+F 0 "#PWR?" H 1400 1800 50  0001 C CNN
+F 1 "+BATT" H 1415 2123 50  0000 C CNN
+F 2 "" H 1400 1950 50  0001 C CNN
+F 3 "" H 1400 1950 50  0001 C CNN
+	1    1400 1950
+	1    0    0    -1
+$EndComp
+$Comp
+L power:PWR_FLAG #FLG?
+U 1 1 5CD8A1D6
+P 1400 2250
+F 0 "#FLG?" H 1400 2325 50  0001 C CNN
+F 1 "PWR_FLAG" H 1400 2423 50  0000 C CNN
+F 2 "" H 1400 2250 50  0001 C CNN
+F 3 "~" H 1400 2250 50  0001 C CNN
+	1    1400 2250
+	-1   0    0    1
+$EndComp
+Wire Wire Line
+	1400 2250 1400 1950
 $EndSCHEMATC

Commit message: description and small changes to schematic
Parts:
- SW2: renamed from SW?; value SW_SPDT -> POWER_SW
- gave numbers to parts that had none: 23

Commit message: added some footprints and edgees for little chassis
Parts:
- removed J4: goldpin 1x2, symbol Connector:Conn_01x02_Female
- added R4: 1,5k, Resistor_SMD:R_0805_2012Metric_Pad1.15x1.40mm_HandSolder, symbol Device:R
- C1, C2, C4, C5, R2, R3: footprint (none) -> Resistor_SMD:R_0805_2012Metric_Pad1.15x1.40mm_HandSolder
- C3, R1: footprint (none) -> Resistor_SMD:R_1206_3216Metric_Pad1.42x1.75mm_HandSolder
- D1, D2: footprint (none) -> LED_SMD:LED_0805_2012Metric_Pad1.15x1.40mm_HandSolder
- D3, D4: footprint (none) -> Diode_SMD:D_SOT-23_NKA; symbol Device:D_Schottky -> Device:D_Schottky_AAK
- D5: footprint (none) -> Diode_SMD:D_SMC_Handsoldering
- J1: value goldpin 1x4 -> goldpin 1x6; footprint (none) -> Connector_PinHeader_2.54mm:PinHeader_1x06_P2.54mm_Horizontal; symbol Connector:Conn_01x04_Male -> Connector:Conn_01x06_Male
- J2: footprint (none) -> Connector_PinHeader_2.54mm:PinHeader_1x02_P2.54mm_Horizontal
- J3: footprint (none) -> Connector_PinHeader_2.54mm:PinHeader_1x01_P2.54mm_Horizontal
- Y1: footprint (none) -> Crystal:Crystal_SMD_HC49-SD_HandSoldering
Connections:
- net +5V: now also J1.6 (Pin_6)
- net GND: now also J1.1 (Pin_1), M1.2 (-)
- net ~RESET: now also J1.5 (Pin_5); no longer J1.4 (Pin_4)
- net at U1.3 (PB7): now also J1.2 (Pin_2); no longer J1.1 (Pin_1)
- net at U1.2 (PB6): now also J1.3 (Pin_3); no longer J1.2 (Pin_2)
- net at U1.1 (PB5): now also J1.4 (Pin_4); no longer J1.3 (Pin_3)
- net at Q1.1 (B): now also R4.1; no longer U1.32 (PA5)
- net at Q1.2 (C): now also D3.1 (A); no longer D3.2 (A)
- net at D4.2 (A): no longer D3.1 (K)
- net M+: now reaches D5.1 (K), J3.2 (Pin_2)
- net M+: now also D4.3 (K), M1.1 (+); no longer D4.1 (K)
- new net: D3.3 (K), D4.1 (A)
- new net: R4.2, U1.32 (PA5)
- no-connect marks 23 -> 26
Changed lines of the file:
@@
 F 0 "R1" V 3407 2350 50  0000 C CNN
 F 1 "10k" V 3200 2350 50  0000 C CNN
-F 2 "" V 3130 2350 50  0001 C CNN
+F 2 "Resistor_SMD:R_1206_3216Metric_Pad1.42x1.75mm_HandSolder" V 3130 2350 50  0001 C CNN
 F 3 "~" H 3200 2350 50  0001 C CNN
 	1    3200 2350
@@
 F 0 "Y1" V 3900 2850 50  0000 L CNN
 F 1 "8MHz" V 4400 2800 50  0000 L CNN
-F 2 "" H 4150 2850 50  0001 C CNN
+F 2 "Crystal:Crystal_SMD_HC49-SD_HandSoldering" H 4150 2850 50  0001 C CNN
 F 3 "~" H 4150 2850 50  0001 C CNN
 	1    4150 2850
@@
 F 0 "C1" V 4000 2550 50  0000 C CNN
 F 1 "22p" V 4000 2800 50  0000 C CNN
-F 2 "" H 3888 2550 50  0001 C CNN
+F 2 "Resistor_SMD:R_0805_2012Metric_Pad1.15x1.40mm_HandSolder" H 3888 2550 50  0001 C CNN
 F 3 "~" H 3850 2700 50  0001 C CNN
 	1    3850 2700
@@
 F 0 "C2" V 3700 2900 50  0000 C CNN
 F 1 "22p" V 3700 3050 50  0000 C CNN
-F 2 "" H 3888 2850 50  0001 C CNN
+F 2 "Resistor_SMD:R_0805_2012Metric_Pad1.15x1.40mm_HandSolder" H 3888 2850 50  0001 C CNN
 F 3 "~" H 3850 3000 50  0001 C CNN
 	1    3850 3000
@@
 F 0 "C4" H 5250 1850 50  0000 C CNN
 F 1 "100n" H 5250 1650 50  0000 C CNN
-F 2 "" H 5388 1600 50  0001 C CNN
+F 2 "Resistor_SMD:R_0805_2012Metric_Pad1.15x1.40mm_HandSolder" H 5388 1600 50  0001 C CNN
 F 3 "~" H 5350 1750 50  0001 C CNN
 	1    5350 1750
@@
 F 0 "C5" H 5550 1850 50  0000 C CNN
 F 1 "100n" H 5550 1650 50  0000 C CNN
-F 2 "" H 5688 1600 50  0001 C CNN
+F 2 "Resistor_SMD:R_0805_2012Metric_Pad1.15x1.40mm_HandSolder" H 5688 1600 50  0001 C CNN
 F 3 "~" H 5650 1750 50  0001 C CNN
 	1    5650 1750
@@
 F 0 "C3" H 5050 1650 50  0000 R CNN
 F 1 "22u" H 5050 1850 50  0000 R CNN
-F 2 "" H 4938 1600 50  0001 C CNN
+F 2 "Resistor_SMD:R_1206_3216Metric_Pad1.42x1.75mm_HandSolder" H 4938 1600 50  0001 C CNN
 F 3 "~" H 4900 1750 50  0001 C CNN
 	1    4900 1750
@@
 	5250 1950 5150 1950
 $Comp
-L Connector:Conn_01x04_Male J1
+L Connector:Conn_01x06_Male J1
 U 1 1 5C46621E
 P 6250 3850
 F 0 "J1" H 6223 3730 50  0000 R CNN
-F 1 "goldpin 1x4" H 6223 3821 50  0000 R CNN
-F 2 "" H 6250 3850 50  0001 C CNN
+F 1 "goldpin 1x6" H 6223 3821 50  0000 R CNN
+F 2 "Connector_PinHeader_2.54mm:PinHeader_1x06_P2.54mm_Horizontal" H 6250 3850 50  0001 C CNN
 F 3 "~" H 6250 3850 50  0001 C CNN
 	1    6250 3850
@@
 Wire Wire Line
 	3450 1950 3450 2350
-Text Label 6200 3400 0    50   ~ 0
+Text Label 6100 3350 0    50   ~ 0
 ~RESET
 Wire Wire Line
-	6200 3400 6000 3400
-Wire Wire Line
-	6000 3400 6000 3650
-Wire Wire Line
-	6000 3650 6050 3650
+	6200 3350 5900 3350
+Wire Wire Line
+	5900 3350 5900 3650
+Wire Wire Line
+	5900 3650 6050 3650
 $Comp
 L Device:LED D1
@@
 F 0 "D1" H 6250 2750 50  0000 C CNN
 F 1 "LED" H 6450 2750 50  0000 C CNN
-F 2 "" H 6250 2850 50  0001 C CNN
+F 2 "LED_SMD:LED_0805_2012Metric_Pad1.15x1.40mm_HandSolder" H 6250 2850 50  0001 C CNN
 F 3 "~" H 6250 2850 50  0001 C CNN
 	1    6250 2850
@@
 F 0 "D2" H 6150 3200 50  0000 C CNN
 F 1 "LED" H 6400 3200 50  0000 C CNN
-F 2 "" H 6250 3050 50  0001 C CNN
+F 2 "LED_SMD:LED_0805_2012Metric_Pad1.15x1.40mm_HandSolder" H 6250 3050 50  0001 C CNN
 F 3 "~" H 6250 3050 50  0001 C CNN
 	1    6250 3050
@@
 F 0 "R2" V 6750 2950 50  0000 C CNN
 F 1 "370" V 6650 2850 50  0000 C CNN
-F 2 "" V 6580 2850 50  0001 C CNN
+F 2 "Resistor_SMD:R_0805_2012Metric_Pad1.15x1.40mm_HandSolder" V 6580 2850 50  0001 C CNN
 F 3 "~" H 6650 2850 50  0001 C CNN
 	1    6650 2850
@@
 F 0 "R3" V 6550 3150 50  0000 C CNN
 F 1 "370" V 6650 3050 50  0000 C CNN
-F 2 "" V 6580 3050 50  0001 C CNN
+F 2 "Resistor_SMD:R_0805_2012Metric_Pad1.15x1.40mm_HandSolder" V 6580 3050 50  0001 C CNN
 F 3 "~" H 6650 3050 50  0001 C CNN
 	1    6650 3050
@@
 	7700 2200 7700 2450
 $Comp
-L Device:D_Schottky D3
+L Device:D_Schottky_AAK D3
 U 1 1 5C472630
 P 7700 3250
 F 0 "D3" V 7746 3171 50  0000 R CNN
 F 1 "D_Schottky" V 7655 3171 50  0000 R CNN
-F 2 "" H 7700 3250 50  0001 C CNN
+F 2 "Diode_SMD:D_SOT-23_NKA" H 7700 3250 50  0001 C CNN
 F 3 "~" H 7700 3250 50  0001 C CNN
 	1    7700 3250
 	0    -1   -1   0
 $EndComp
-Wire Wire Line
-	7700 3100 7700 2850
-$Comp
-L Device:D_Schottky D4
+$Comp
+L Device:D_Schottky_AAK D4
 U 1 1 5C473502
 P 7700 3700
 F 0 "D4" V 7746 3621 50  0000 R CNN
 F 1 "D_Schottky" V 7655 3621 50  0000 R CNN
-F 2 "" H 7700 3700 50  0001 C CNN
+F 2 "Diode_SMD:D_SOT-23_NKA" H 7700 3700 50  0001 C CNN
 F 3 "~" H 7700 3700 50  0001 C CNN
 	1    7700 3700
 	0    -1   -1   0
 $EndComp
-Wire Wire Line
-	7700 3550 7700 3400
 $Comp
 L Device:D D5
@@
 F 0 "D5" V 7654 4229 50  0000 L CNN
 F 1 "D" V 7745 4229 50  0000 L CNN
-F 2 "" H 7700 4150 50  0001 C CNN
+F 2 "Diode_SMD:D_SMC_Handsoldering" H 7700 4150 50  0001 C CNN
 F 3 "~" H 7700 4150 50  0001 C CNN
 	1    7700 4150
@@
 P 8300 4200
 F 0 "J3" H 8406 4378 50  0000 C CNN
-F 1 "goldpin 1x2" H 8300 3950 50  0000 C CNN
-F 2 "" H 8300 4200 50  0001 C CNN
+F 1 "goldpin 1x2" H 8200 4450 50  0000 C CNN
+F 2 "Connector_PinHeader_2.54mm:PinHeader_1x01_P2.54mm_Horizontal" H 8300 4200 50  0001 C CNN
 F 3 "~" H 8300 4200 50  0001 C CNN
 	1    8300 4200
@@
 F 0 "J2" H 6310 5190 50  0000 L CNN
 F 1 "goldpin 1x2" H 6150 5300 50  0000 L CNN
-F 2 "" H 6250 5150 50  0001 C CNN
+F 2 "Connector_PinHeader_2.54mm:PinHeader_1x02_P2.54mm_Horizontal" H 6250 5150 50  0001 C CNN
 F 3 "~" H 6250 5150 50  0001 C CNN
 	1    6250 5150
@@
 U 1 1 5C49ECC9
 P 6450 2350
-F 0 "SW3" H 6500 2500 50  0000 R CNN
-F 1 "ACTION SW" H 6600 2250 50  0000 R CNN
+F 0 "SW3" H 6550 2600 50  0000 R CNN
+F 1 "ACTION SW" H 6700 2500 50  0000 R CNN
 F 2 "" H 6450 2350 50  0001 C CNN
 F 3 "" H 6450 2350 50  0001 C CNN
@@
 	1    0    0    -1
 $EndComp
-Wire Wire Line
-	5850 2650 7400 2650
 Text Notes 8300 3600 0    50   ~ 0
 Silnik\nwibracyjny
@@
 	8000 3950 8000 4100
 Wire Wire Line
-	8000 4100 8100 4100
-Wire Wire Line
-	8000 4200 8100 4200
+	8000 4200 8050 4200
 $Comp
 L Motor:Motor_DC M1
@@
 	1    0    0    -1
 $EndComp
-$Comp
-L Connector:Conn_01x02_Female J4
-U 1 1 5CD5CD44
-P 8500 4200
-F 0 "J4" H 8394 3875 50  0000 C CNN
-F 1 "goldpin 1x2" H 8400 4300 50  0000 C CNN
-F 2 "" H 8500 4200 50  0001 C CNN
-F 3 "~" H 8500 4200 50  0001 C CNN
-	1    8500 4200
-	-1   0    0    1
-$EndComp
 Wire Wire Line
 	9100 4350 9100 4400
@@
 	8850 4200 8700 4200
 Wire Wire Line
-	8700 4100 8850 4100
-Wire Wire Line
 	8850 4100 8850 3800
 Wire Wire Line
@@
 	5850 3250 6950 3250
 Wire Notes Line
-	6950 3250 6950 4150
-Wire Notes Line
-	6950 4150 5850 4150
-Wire Notes Line
-	5850 4150 5850 3250
-Text Notes 6550 4000 0    50   ~ 0
+	6950 3250 6950 4350
+Wire Notes Line
+	5850 4350 5850 3250
+Text Notes 6550 3600 0    50   ~ 0
 USBasp
 $Comp
@@
 Wire Wire Line
 	1400 2250 1400 1950
+NoConn ~ 4550 2950
+Wire Wire Line
+	5950 3450 5950 3550
+Wire Wire Line
+	5950 3550 6050 3550
+Text Label 6350 3450 0    50   ~ 0
++5V_USBasp
+Wire Notes Line
+	5850 4350 6950 4350
+Text Label 4850 1300 0    50   ~ 0
++5V_USBasp
+Wire Wire Line
+	4500 1350 4850 1350
+Wire Wire Line
+	4850 1350 4850 1300
+Connection ~ 4500 1350
+$Comp
+L power:GND #PWR0101
+U 1 1 5CDFCCDD
+P 6000 4100
+F 0 "#PWR0101" H 6000 3850 50  0001 C CNN
+F 1 "GND" H 6005 3927 50  0000 C CNN
+F 2 "" H 6000 4100 50  0001 C CNN
+F 3 "" H 6000 4100 50  0001 C CNN
+	1    6000 4100
+	1    0    0    -1
+$EndComp
+Wire Wire Line
+	5950 3450 6350 3450
+Wire Wire Line
+	6000 4100 6000 4050
+Wire Wire Line
+	6000 4050 6050 4050
+$Comp
+L Device:R R4
+U 1 1 5CE05FB9
+P 6450 2650
+F 0 "R4" V 6350 2650 50  0000 C CNN
+F 1 "1,5k" V 6450 2650 50  0000 C CNN
+F 2 "Resistor_SMD:R_0805_2012Metric_Pad1.15x1.40mm_HandSolder" V 6380 2650 50  0001 C CNN
+F 3 "~" H 6450 2650 50  0001 C CNN
+	1    6450 2650
+	0    1    1    0
+$EndComp
+Wire Wire Line
+	5850 2650 6300 2650
+Wire Wire Line
+	6600 2650 7400 2650
+Wire Wire Line
+	7600 3050 7600 2950
+Wire Wire Line
+	7600 2950 7700 2950
+Wire Wire Line
+	7700 2950 7700 2850
+Wire Wire Line
+	7600 3500 7600 3450
+Wire Wire Line
+	7600 3450 7700 3450
+Wire Wire Line
+	7700 3450 7700 3400
+NoConn ~ 7700 3500
+NoConn ~ 7700 3050
+Text Label 8700 4100 2    50   ~ 0
+M+
+Text Label 8700 4200 2    50   ~ 0
+M-
+Wire Wire Line
+	8700 4100 8850 4100
+Wire Wire Line
+	8000 4100 8050 4100
+Wire Wire Line
+	8050 4100 8050 3950
+Wire Wire Line
+	8050 3950 8700 3950
+Wire Wire Line
+	8700 3950 8700 4100
+Connection ~ 8050 4100
+Wire Wire Line
+	8050 4100 8100 4100
+Wire Wire Line
+	8050 4200 8050 4300
+Wire Wire Line
+	8050 4300 8700 4300
+Wire Wire Line
+	8700 4300 8700 4200
+Connection ~ 8050 4200
+Wire Wire Line
+	8050 4200 8100 4200
 $EndSCHEMATC

Commit message: added few footprints and created two pcb boards WIP
Parts:
- J3: footprint Connector_PinHeader_2.54mm:PinHeader_1x01_P2.54mm_Horizontal -> Connector_PinHeader_2.54mm:PinHeader_1x02_P2.54mm_Horizontal
- Q1: footprint (none) -> Package_TO_SOT_SMD:SOT-223
- SW1: footprint (none) -> MyFootprints:MYSMDSWITCH
- SW2: footprint (none) -> MyFootprints:MYSUWAKSMDSWITCH
- SW3: footprint (none) -> MyFootprints:MYSWITCHWITHLEWER
Changed lines of the file:
@@
 F 0 "SW1" V 3500 3100 50  0000 R CNN
 F 1 "RESET SW" V 3350 3200 50  0000 R CNN
-F 2 "" H 3450 2750 50  0001 C CNN
+F 2 "MyFootprints:MYSMDSWITCH" H 3450 2750 50  0001 C CNN
 F 3 "" H 3450 2750 50  0001 C CNN
 	1    3450 2750
@@
 F 0 "Q1" H 7791 2604 50  0000 L CNN
 F 1 "Q_PNP_BCE" H 7791 2695 50  0000 L CNN
-F 2 "" H 7800 2750 50  0001 C CNN
+F 2 "Package_TO_SOT_SMD:SOT-223" H 7800 2750 50  0001 C CNN
 F 3 "~" H 7600 2650 50  0001 C CNN
 	1    7600 2650
@@
 F 0 "J3" H 8406 4378 50  0000 C CNN
 F 1 "goldpin 1x2" H 8200 4450 50  0000 C CNN
-F 2 "Connector_PinHeader_2.54mm:PinHeader_1x01_P2.54mm_Horizontal" H 8300 4200 50  0001 C CNN
+F 2 "Connector_PinHeader_2.54mm:PinHeader_1x02_P2.54mm_Horizontal" H 8300 4200 50  0001 C CNN
 F 3 "~" H 8300 4200 50  0001 C CNN
 	1    8300 4200
@@
 F 0 "SW3" H 6550 2600 50  0000 R CNN
 F 1 "ACTION SW" H 6700 2500 50  0000 R CNN
-F 2 "" H 6450 2350 50  0001 C CNN
+F 2 "MyFootprints:MYSWITCHWITHLEWER" H 6450 2350 50  0001 C CNN
 F 3 "" H 6450 2350 50  0001 C CNN
 	1    6450 2350
@@
 F 0 "SW2" V 4350 1900 50  0000 R CNN
 F 1 "POWER_SW" V 4250 2000 50  0000 R CNN
-F 2 "" H 4400 1550 50  0001 C CNN
+F 2 "MyFootprints:MYSUWAKSMDSWITCH" H 4400 1550 50  0001 C CNN
 F 3 "" H 4400 1550 50  0001 C CNN
 	1    4400 1550

Commit message: pcb in progress
Parts:
- added J4: goldpin 1x2, Connector_PinHeader_2.54mm:PinHeader_1x02_P2.54mm_Horizontal, symbol Connector:Conn_01x02_Male
- D3, D4: footprint Diode_SMD:D_SOT-23_NKA -> Package_TO_SOT_SMD:SOT-23_Handsoldering
Connections:
- net +BATT: now also J4.2 (Pin_2)
- net GND: now also J1.6 (Pin_6), J4.1 (Pin_1); no longer J1.1 (Pin_1)
- net M+: now also D3.3 (K); no longer D4.3 (K)
- net ~RESET: now also J1.1 (Pin_1); no longer J1.5 (Pin_5)
- net VCC: now reaches C3.1, C4.2, C5.2, SW2.2 (B), U1.17 (VCC), U1.27 (AVCC), U1.38 (VCC), U1.5 (VCC)
- net VCC: now also Q1.3 (E), R1.1
- net at Q1.2 (C): now also D4.1 (A); no longer D3.1 (A)
- net at SW3.1 (A): now also U1.12 (PD3); no longer U1.36 (PA1)
- removed net +5V: J1.6 (Pin_6), Q1.3 (E), R1.1, SW2.3 (C)
- new net: D3.1 (A), D4.3 (K)
- new net +5V_USBasp: J1.5 (Pin_5), SW2.3 (C)
Other:
- moved on the sheet: C1, D3, D4, J2, SW2, SW3A, Y1

Commit message: zrzut
Parts:
- removed D3, D4: D_Schottky, Package_TO_SOT_SMD:SOT-23_Handsoldering, symbol Device:D_Schottky_AAK
- removed J4: goldpin 1x2, Connector_PinHeader_2.54mm:PinHeader_1x02_P2.54mm_Horizontal, symbol Connector:Conn_01x02_Male
- removed SW2: POWER_SW, MyFootprints:MYSUWAKSMDSWITCH, symbol Switch:SW_SPDT
- added R5, R6: 10k, Resistor_SMD:R_1206_3216Metric_Pad1.42x1.75mm_HandSolder, symbol Device:R
- Q1: value Q_PNP_BCE -> PNP
- R4: value 1,5k -> 4k
- SW1: footprint MyFootprints:MYSMDSWITCH -> Button_Switch_SMD:SW_SPST_EVQPE1
- SW3: value ACTION SW -> LEVER_SW
Connections:
- net +5V_USBasp is gone; now on net VCC: J1.5 (Pin_5)
- net GND: now also J3.2 (Pin_2), R6.2; no longer J3.1 (Pin_1)
- net VCC: now also Q1.2 (C), R5.1; no longer Q1.3 (E)
- net at SW3.1 (A): now also U1.11 (PD2); no longer U1.12 (PD3)
- net PWM_M: now reaches U1.14 (PD5)
- net PWM_M: now also R4.2
- net at U1.32 (PA5): no longer R4.2
- net VCC_half: now reaches U1.36 (PA1)
- net VCC_half: now also R5.2, R6.1
- net M+: no longer names the net of D5.1 (K), M1.1 (+)
- net M+: now also J3.1 (Pin_1), Q1.3 (E); no longer J3.2 (Pin_2)
- no-connect marks 26 -> 23
Other:
- moved on the sheet: D1, D2, D5, J2, J3, M1, Q1, R2, R3, R4, SW3A

Commit message: Przygotowanie plikow do wytrawiania plytki
Connections:
- net M+: now reaches D5.1 (K), J3.1 (Pin_1), M1.1 (+), Q1.3 (E)
Other:
- moved on the sheet: J3
Changed lines of the file:
@@
 U 1 1 5C474305
 P 8550 3350
-F 0 "D5" V 8504 3429 50  0000 L CNN
-F 1 "D" V 8595 3429 50  0000 L CNN
+F 0 "D5" V 8450 3150 50  0000 L CNN
+F 1 "D" V 8600 3150 50  0000 L CNN
 F 2 "Diode_SMD:D_SMC_Handsoldering" H 8550 3350 50  0001 C CNN
 F 3 "~" H 8550 3350 50  0001 C CNN
@@
 F 3 "" H 8550 3600 50  0001 C CNN
 	1    8550 3600
-	1    0    0    -1
-$EndComp
-$Comp
-L Connector:Conn_01x02_Male J3
-U 1 1 5C478F49
-P 8950 3300
-F 0 "J3" H 9000 3400 50  0000 C CNN
-F 1 "goldpin 1x2" H 9900 4450 50  0001 C CNN
-F 2 "Connector_PinHeader_2.54mm:PinHeader_1x02_P2.54mm_Horizontal" H 8950 3300 50  0001 C CNN
-F 3 "~" H 8950 3300 50  0001 C CNN
-	1    8950 3300
 	1    0    0    -1
 $EndComp
@@
 	6500 3400 6500 3350
 Wire Wire Line
-	9150 3100 9500 3100
-Wire Wire Line
-	9150 3600 9500 3600
-Wire Wire Line
-	8550 2900 8550 3100
-Wire Wire Line
-	9150 3100 9150 3300
-Wire Wire Line
 	8550 3500 8550 3600
-Wire Wire Line
-	9150 3400 9150 3600
-Wire Wire Line
-	8550 3100 9150 3100
-Connection ~ 9150 3100
-Connection ~ 8550 3100
-Wire Wire Line
-	8550 3100 8550 3200
-Wire Wire Line
-	9150 3600 8550 3600
-Connection ~ 9150 3600
-Connection ~ 8550 3600
 Wire Wire Line
 	8200 2700 8250 2700
@@
 	6850 2650 6850 2850
 Connection ~ 6850 2850
+Wire Wire Line
+	8550 2900 8550 3200
+Wire Wire Line
+	9500 3600 9300 3600
+Wire Wire Line
+	9500 3100 9300 3100
+Text Label 9300 3100 2    50   ~ 0
+M+
+Text Label 9300 3600 2    50   ~ 0
+M-
+Connection ~ 8550 3500
+Connection ~ 8550 3200
+$Comp
+L Connector:Conn_01x02_Male J3
+U 1 1 5C478F49
+P 8750 3300
+F 0 "J3" H 8650 3250 50  0000 C CNN
+F 1 "goldpin 1x2" H 9700 4450 50  0001 C CNN
+F 2 "Connector_PinHeader_2.54mm:PinHeader_1x02_P2.54mm_Horizontal" H 8750 3300 50  0001 C CNN
+F 3 "~" H 8750 3300 50  0001 C CNN
+	1    8750 3300
+	1    0    0    -1
+$EndComp
+Wire Wire Line
+	8950 3500 8950 3400
+Wire Wire Line
+	8550 3500 8950 3500
+Wire Wire Line
+	8950 3200 8950 3300
+Wire Wire Line
+	8550 3200 8950 3200
+Text Label 8950 3300 0    50   ~ 0
+M+
+Text Label 8950 3400 0    50   ~ 0
+M-
 $EndSCHEMATC
